Commit message: launch fixes

File: ros_ws/src/robot_urdf/urdf_model/robot.urdf (robot description, URDF)
Before this commit: robot basic_mobile_bot, 5 links, 4 joints
Links:
- removed link lidar_link
- added link base_laser; visual mesh filename=package://robot_urdf/meshes/lidar.stl scale=0.001 0.001 0.001
Joints:
- joint lidar_joint: child lidar_link -> base_laser

Commit message: simplifying config and launch, adding cliff sensor(not working yet)

File: ros_ws/src/robot_urdf/urdf_model/robot.urdf (robot description, URDF)
Before this commit: robot basic_mobile_bot, 5 links, 4 joints
Links:
- added link base_cliff_sensor; visual box size=0.03 0.02 0.01
Joints:
- added joint base_cliff_sensor_joint: type fixed, parent base_link, child base_cliff_sensor, origin xyz=0.08 0 0.005 rpy=0 0 ${pi/2}
- joint caster_joint: origin xyz=${caster_xoff} 0.0 -0.0294 rpy=0 0 0 -> xyz=${caster_xoff} 0.0 0.0106 rpy=0 0 0

Commit message: ultrasonic sensor

File: ros_ws/src/robot_urdf/urdf_model/robot.urdf (robot description, URDF)
Before this commit: robot basic_mobile_bot, 6 links, 5 joints
Joints:
- joint base_cliff_sensor_joint: origin xyz=0.08 0 0.005 rpy=0 0 ${pi/2} -> xyz=0.09 0 0.045 rpy=0 0 0
- joint lidar_joint: origin xyz=0.011 0 0.0864 rpy=0 0 ${pi/2} -> xyz=0.011 0 0.1264 rpy=0 0 ${pi/2}
